File: PCB/QMTECH/ospi.kicad_pcb (KiCad board)
At the start: 2 copper layers, 67.1 x 88.9 mm, 50 parts, among them J1 USB_C_Receptacle_Power, J10 Conn_02x06_Odd_Even, J2 Conn_01x06_Male, J3 Conn_02x07_Odd_Even, J4 Conn_02x32_Odd_Even, J5 Conn_02x22_Odd_Even, J6 USB_C_Receptacle_8pin, J7 Conn_02x22_Odd_Even, J8 Conn_01x32_Male, J9 Conn_02x06_Odd_Even, SW1 SW_Push, U1 USB3300-EZK, Y1 Crystal_GND24

Commit message: PCB更新
Parts:
- C5, C8: moved to B.Cu
- U1: footprint Package_DFN_QFN:QFN-32-1EP_5x5mm_P0.5mm_EP3.45x3.45mm -> My:QFN-32-1EP_5x5mm_P0.5mm_EP3.45x3.45mm_ThermalVias
- moved R18 8.80 mm to (105.9, 57.7), turned to -90 degrees
- moved C8 2.55 mm to (113.8, 48.3), turned to -90 degrees
- moved R1 2.19 mm to (124.4, 55.4), turned to 180 degrees
- moved R2 1.67 mm to (130.2, 55.4), turned to 0 degrees
- moved C5 1.50 mm to (111.0, 48.3), turned to -90 degrees
Routing:
- net +5VD: track 18.7 -> 4.47 mm
- net GND: track 502.6 -> 511.2 mm
- net VBUS: track 49.4 -> 53.6 mm
- net Net-(J1-PadB5): track 4.15 -> 7.05 mm
- net Net-(J1-PadA5): track 4.46 -> 6.97 mm
Other:
- board text added: "Rev. A.2"
- board text removed: "Rev. A"
