File: PCB/QMTECH/ospi.kicad_sch (KiCad schematic)
At the start: 50 parts, among them J1 USB_C_Receptacle_Power, J10 Conn_02x06_Odd_Even, J2 Conn_01x06_Male, J3 Conn_02x07_Odd_Even, J4 Conn_02x32_Odd_Even, J5 Conn_02x22_Odd_Even, J6 USB_C_Receptacle_8pin, J7 Conn_02x22_Odd_Even, J8 Conn_01x32_Male, J9 Conn_02x06_Odd_Even, SW1 SW_Push, U1 USB3300-EZK, Y1 Crystal_GND24

Commit message: PCB更新
Parts:
- U1: footprint Package_DFN_QFN:QFN-32-1EP_5x5mm_P0.5mm_EP3.45x3.45mm -> My:QFN-32-1EP_5x5mm_P0.5mm_EP3.45x3.45mm_ThermalVias
Changed lines of the file:
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@@
     (property "Reference" "U1" (id 0) (at 168.275 44.2212 90))
     (property "Value" "USB3300-EZK" (id 1) (at 168.275 46.7612 90))
-    (property "Footprint" "Package_DFN_QFN:QFN-32-1EP_5x5mm_P0.5mm_EP3.45x3.45mm" (id 2) (at 169.545 86.36 0)
+    (property "Footprint" "My:QFN-32-1EP_5x5mm_P0.5mm_EP3.45x3.45mm_ThermalVias" (id 2) (at 169.545 86.36 0)
       (effects (font (size 1.27 1.27)) hide)
     )
@@
     )
     (path "/ae45b09c-78e3-44d1-9f74-a1c80ff1dd73"
-      (reference "U1") (unit 1) (value "USB3300-EZK") (footprint "Package_DFN_QFN:QFN-32-1EP_5x5mm_P0.5mm_EP3.45x3.45mm")
+      (reference "U1") (unit 1) (value "USB3300-EZK") (footprint "My:QFN-32-1EP_5x5mm_P0.5mm_EP3.45x3.45mm_ThermalVias")
     )
     (path "/5b82de44-5dfc-40a7-a488-13883d03244c"
